Commit message: ロボットからLRFが落ちた

File: dual_lidar_robot/urdf/move_lrf_robot.urdf (robot description, URDF)
Before this commit: robot my_robo, 7 links, 6 joints
Joints:
- joint hokuyo_joint_back: type fixed -> floating
- joint hokuyo_joint_front: type fixed -> floating

Commit message: 落ちないようにした

File: dual_lidar_robot/urdf/move_lrf_robot.urdf (robot description, URDF)
Before this commit: robot my_robo, 7 links, 6 joints
Joints:
- joint hokuyo_joint_back: axis 0 1 0 -> 0 0 1; limit (none) -> lower=0 upper=10.0 effort=0 velocity=1.0; type floating -> prismatic
- joint hokuyo_joint_front: axis 0 1 0 -> 0 0 1; limit (none) -> lower=0 upper=10.0 effort=0 velocity=1.0; type floating -> prismatic
